Commit message: add gazebo and rviz description

File: robots/kobuki_description/urdf/kobuki.urdf.xacro (robot description, xacro)
@@ -7,6 +7,6 @@
  -->
 <robot name="kobuki" xmlns:xacro="http://ros.org/wiki/xacro">
-  <xacro:include filename="$(find kobuki_description)/urdf/common_properties.urdf.xacro"/>
-  <xacro:include filename="$(find kobuki_description)/urdf/kobuki_gazebo.urdf.xacro"/>
+  <xacro:include filename="$(find butler)/robots/kobuki_description/urdf/common_properties.urdf.xacro"/>
+  <xacro:include filename="$(find butler)/robots/kobuki_description/urdf/kobuki_gazebo.urdf.xacro"/>
   <!-- Kobuki -->
   <xacro:macro name="kobuki">
@@ -30,5 +30,5 @@
         <geometry>
           <!-- new mesh -->
-          <mesh filename="package://kobuki_description/meshes/main_body.dae" />
+          <mesh filename="package://butler/robots/kobuki_description/meshes/main_body.dae" />
         </geometry>
         <origin xyz="0.001 0 0.05199" rpy="0 0 0"/>
@@ -65,5 +65,5 @@
       <visual>
         <geometry>
-          <mesh filename="package://kobuki_description/meshes/wheel.dae"/>
+          <mesh filename="package://butler/robots/kobuki_description/meshes/wheel.dae"/>
         </geometry>
         <origin xyz="0 0 0" rpy="0 0 0"/>
@@ -92,5 +92,5 @@
       <visual>
         <geometry>
-          <mesh filename="package://kobuki_description/meshes/wheel.dae"/>
+          <mesh filename="package://butler/robots/kobuki_description/meshes/wheel.dae"/>
         </geometry>
         <origin xyz="0 0 0" rpy="0 0 0"/>

File: robots/kobuki_description/urdf/kobuki_standalone.urdf.xacro (robot description, xacro)
@@ -1,4 +1,4 @@
 <?xml version="1.0"?>
-<robot name="kobuki_standalone"
+<robot name="kobuki"
        xmlns:sensor="http://playerstage.sourceforge.net/gazebo/xmlschema/#sensor"
        xmlns:controller="http://playerstage.sourceforge.net/gazebo/xmlschema/#controller"
@@ -6,5 +6,5 @@
        xmlns:xacro="http://ros.org/wiki/xacro">
   <!-- Defines the kobuki component tag. -->
-  <xacro:include filename="$(find kobuki_description)/urdf/kobuki.urdf.xacro" />
+  <xacro:include filename="$(find butler)/robots/kobuki_description/urdf/kobuki.urdf.xacro" />
   <kobuki/>
 </robot>
