Commit message: Added yaml parameter parsing

File: robots/jackal_description/urdf/accessories.urdf.xacro (robot description, xacro)
@@ -9,4 +9,24 @@
     jackal_base/launch/base.launch
   -->
+  <!-- Macro to read in parameters from yaml file. -->
+  <xacro:macro name="read_model_data" params="config_jackal_file">
+    <xacro:property name="__LASER" value="${config_jackal_file['LASER']}"/>
+    <xacro:property name="__NAVSAT" value="${config_jackal_file['NAVSAT']}"/>
+    <xacro:property name="__FENDER" value="${config_jackal_file['FENDER']}"/>
+    <xacro:property name="__JACKAL_ARC_ENCLOSURE" value="${config_jackal_file['JACKAL_ARC_ENCLOSURE']}"/>
+    <xacro:property name="jackal_laser" value="${__LASER['JACKAL_LASER']}" scope="parent"/>
+    <xacro:property name="jackal_laser_hokuyo" value="${__LASER['JACKAL_LASER_HOKUYO']}" scope="parent"/>
+    <xacro:property name="jackal_laser_mount" value="${__LASER['JACKAL_LASER_MOUNT']}" scope="parent"/>
+    <xacro:property name="jackal_laser_topic" value="${__LASER['JACKAL_LASER_TOPIC']}" scope="parent"/>
+    <xacro:property name="jackal_laser_offset" value="${__LASER['JACKAL_LASER_OFFSET']}" scope="parent"/>
+    <xacro:property name="jackal_laser_rpy" value="${__LASER['JACKAL_LASER_RPY']}" scope="parent"/>
+    <xacro:property name="jackal_navsat" value="${__NAVSAT['JACKAL_NAVSAT']}" scope="parent"/>
+    <xacro:property name="jackal_navsat_mount" value="${__NAVSAT['JACKAL_NAVSAT_MOUNT']}" scope="parent"/>
+    <xacro:property name="jackal_navsat_height" value="${__NAVSAT['JACKAL_NAVSAT_HEIGHT']}" scope="parent"/>
+    <xacro:property name="jackal_front_accessory_fender" value="${__FENDER['JACKAL_FRONT_ACCESSORY_FENDER']}" scope="parent"/>
+    <xacro:property name="jackal_rear_accessory_fender" value="${__FENDER['JACKAL_REAR_ACCESSORY_FENDER']}" scope="parent"/>
+    <xacro:property name="jackal_front_fender_ust10" value="${__FENDER['JACKAL_FRONT_FENDER_UST10']}" scope="parent"/>
+    <xacro:property name="jackal_rear_fender_ust10" value="${__FENDER['JACKAL_REAR_FENDER_UST10']}" scope="parent"/>
+  </xacro:macro>
   <!-- Macros to generate standoffs for offset payload mounting. -->
   <xacro:include filename="$(find butler)/robots/jackal_description/urdf/accessories/standoffs.urdf.xacro" />
@@ -14,38 +34,38 @@
   <xacro:include filename="$(find butler)/robots/jackal_description/urdf/accessories/bridge_plate.urdf.xacro" />
   <!-- If enabled, generate the LASER payload (by default, a SICK LMS111). -->
-  <xacro:if value="$(optenv JACKAL_LASER 0)">
-    <xacro:if value="$(optenv JACKAL_LASER_HOKUYO 0)">
+  <xacro:if value="$(jackal_laser == 0)">
+    <xacro:if value="$(jackal_laser_hokuyo == 0)">
       <xacro:include filename="$(find butler)/robots/jackal_description/urdf/accessories/hokuyo_ust10.urdf.xacro" />
-      <hokuyo_ust10_mount prefix="$(optenv JACKAL_LASER_MOUNT front)"
-                          topic="$(optenv JACKAL_LASER_TOPIC front/scan)" />
-      <joint name="$(optenv JACKAL_LASER_MOUNT front)_laser_mount_joint" type="fixed">
-        <origin xyz="$(optenv JACKAL_LASER_OFFSET 0.11 0 0)"
-                rpy="$(optenv JACKAL_LASER_RPY 0 0 0)" />
-        <parent link="$(optenv JACKAL_LASER_MOUNT front)_mount" />
-        <child link="$(optenv JACKAL_LASER_MOUNT front)_laser_mount" />
+      <hokuyo_ust10_mount prefix="$(jackal_laser_mount)"
+                          topic="$(jackal_laser_topic)" />
+      <joint name="$(jackal_laser_mount)_laser_mount_joint" type="fixed">
+        <origin xyz="$(jackal_laser_offset)"
+                rpy="$(jackal_laser_rpy)" />
+        <parent link="$(jackal_laser_mount)_mount" />
+        <child link="$(jackal_laser_mount)_laser_mount" />
       </joint>
     </xacro:if>
-    <xacro:unless value="$(optenv JACKAL_LASER_HOKUYO 0)">
+    <xacro:unless value="$(jackal_laser_hokuyo)">
       <xacro:include filename="$(find butler)/robots/jackal_description/urdf/accessories/sick_lms1xx_mount.urdf.xacro" />
-      <sick_lms1xx_mount prefix="$(optenv JACKAL_LASER_MOUNT front)"
-                         topic="$(optenv JACKAL_LASER_TOPIC front/scan)"/>
-      <joint name="$(optenv JACKAL_LASER_MOUNT front)_laser_mount_joint" type="fixed">
-        <origin xyz="$(optenv JACKAL_LASER_OFFSET 0 0 0)"
-                rpy="$(optenv JACKAL_LASER_RPY 0 0 0)" />
-        <parent link="$(optenv JACKAL_LASER_MOUNT front)_mount" />
-        <child link="$(optenv JACKAL_LASER_MOUNT front)_laser_mount" />
+      <sick_lms1xx_mount prefix="$(jackal_laser_mount)"
+                         topic="$(jackal_laser_topic)"/>
+      <joint name="$(jackal_laser_mount)_laser_mount_joint" type="fixed">
+        <origin xyz="$(jackal_laser_offset)"
+                rpy="$(jackal_laser_rpy)" />
+        <parent link="$(jackal_laser_mount)_mount" />
+        <child link="$(jackal_laser_mount)_laser_mount" />
       </joint>
     </xacro:unless>
   </xacro:if>
   <!-- If enabled, generate the upgraded Navsat payload (a Novatel Smart6). -->
-  <xacro:if value="$(optenv JACKAL_NAVSAT 0)">
+  <xacro:if value="$(jackal_navsat)">
     <xacro:include filename="$(find butler)/robots/jackal_description/urdf/accessories/novatel_smart6.urdf.xacro" />
-    <bridge_plate mount="$(optenv JACKAL_NAVSAT_MOUNT rear)"
-                  height="$(optenv JACKAL_NAVSAT_HEIGHT 0.1)" />
-    <novatel_smart6 prefix="$(optenv JACKAL_NAVSAT_MOUNT rear)"/>
-    <joint name="$(optenv JACKAL_NAVSAT_MOUNT rear)_navsat_joint" type="fixed">
+    <bridge_plate mount="$(jackal_navsat_mount)"
+                  height="$(jackal_navsat_height)" />
+    <novatel_smart6 prefix="$(jackal_navsat_mount)"/>
+    <joint name="$(jackal_navsat_mount)_navsat_joint" type="fixed">
       <origin xyz="0 0 0" rpy="0 0 0" />
-      <parent link="$(optenv JACKAL_NAVSAT_MOUNT rear)_bridge" />
-      <child link="$(optenv JACKAL_NAVSAT_MOUNT rear)_navsat" />
+      <parent link="$(jackal_navsat_mount)_bridge" />
+      <child link="$(jackal_navsat_mount)_navsat" />
     </joint>
   </xacro:if>
@@ -121,16 +141,16 @@
     </joint>
   </xacro:if> -->
-  <xacro:if value="$(optenv JACKAL_FRONT_ACCESSORY_FENDER 0)">
+  <xacro:if value="$(jackal_front_accessory_fender)">
     <xacro:include filename="$(find butler)/robots/jackal_description/urdf/accessories/hokuyo_ust10.urdf.xacro" />
-    <xacro:if value="$(optenv JACKAL_FRONT_FENDER_UST10 0)">
+    <xacro:if value="$(jackal_front_fender_ust10)">
         <hokuyo_ust10 prefix="front_ust10" parent_link="front_fender_accessory_link"/>
     </xacro:if>
   </xacro:if>
-  <xacro:if value="$(optenv JACKAL_REAR_ACCESSORY_FENDER 0)">
-    <xacro:if value="$(optenv JACKAL_REAR_FENDER_UST10 0)">
+  <xacro:if value="$(jackal_rear_accessory_fender)">
+    <xacro:if value="$(jackal_rear_fender_ust10)">
         <hokuyo_ust10 prefix="rear_ust10" parent_link="rear_fender_accessory_link"/>
     </xacro:if>
   </xacro:if>
-  <xacro:if value="$(optenv JACKAL_ARK_ENCLOSURE 0)">
+  <xacro:if value="$(__JACKAL_ARK_ENCLOSURE)">
     <link name="ark_enclosure_link">
       <visual>

Commit message: Updated YAML read

File: robots/jackal_description/urdf/accessories.urdf.xacro (robot description, xacro)
@@ -10,23 +10,7 @@
   -->
   <!-- Macro to read in parameters from yaml file. -->
-  <xacro:macro name="read_model_data" params="config_jackal_file">
-    <xacro:property name="__LASER" value="${config_jackal_file['LASER']}"/>
-    <xacro:property name="__NAVSAT" value="${config_jackal_file['NAVSAT']}"/>
-    <xacro:property name="__FENDER" value="${config_jackal_file['FENDER']}"/>
-    <xacro:property name="__JACKAL_ARC_ENCLOSURE" value="${config_jackal_file['JACKAL_ARC_ENCLOSURE']}"/>
-    <xacro:property name="jackal_laser" value="${__LASER['JACKAL_LASER']}" scope="parent"/>
-    <xacro:property name="jackal_laser_hokuyo" value="${__LASER['JACKAL_LASER_HOKUYO']}" scope="parent"/>
-    <xacro:property name="jackal_laser_mount" value="${__LASER['JACKAL_LASER_MOUNT']}" scope="parent"/>
-    <xacro:property name="jackal_laser_topic" value="${__LASER['JACKAL_LASER_TOPIC']}" scope="parent"/>
-    <xacro:property name="jackal_laser_offset" value="${__LASER['JACKAL_LASER_OFFSET']}" scope="parent"/>
-    <xacro:property name="jackal_laser_rpy" value="${__LASER['JACKAL_LASER_RPY']}" scope="parent"/>
-    <xacro:property name="jackal_navsat" value="${__NAVSAT['JACKAL_NAVSAT']}" scope="parent"/>
-    <xacro:property name="jackal_navsat_mount" value="${__NAVSAT['JACKAL_NAVSAT_MOUNT']}" scope="parent"/>
-    <xacro:property name="jackal_navsat_height" value="${__NAVSAT['JACKAL_NAVSAT_HEIGHT']}" scope="parent"/>
-    <xacro:property name="jackal_front_accessory_fender" value="${__FENDER['JACKAL_FRONT_ACCESSORY_FENDER']}" scope="parent"/>
-    <xacro:property name="jackal_rear_accessory_fender" value="${__FENDER['JACKAL_REAR_ACCESSORY_FENDER']}" scope="parent"/>
-    <xacro:property name="jackal_front_fender_ust10" value="${__FENDER['JACKAL_FRONT_FENDER_UST10']}" scope="parent"/>
-    <xacro:property name="jackal_rear_fender_ust10" value="${__FENDER['JACKAL_REAR_FENDER_UST10']}" scope="parent"/>
-  </xacro:macro>
+  <xacro:include filename="$(find butler)/robots/jackal_description/urdf/jackal.macro.xacro" />
+  <xacro:macro name="jackal" params="prefix config_jackal_file" >
+   <xacro:read_model_data config_jackal_file="${config_jackal_file}"/>
   <!-- Macros to generate standoffs for offset payload mounting. -->
   <xacro:include filename="$(find butler)/robots/jackal_description/urdf/accessories/standoffs.urdf.xacro" />
@@ -39,12 +23,12 @@
       <hokuyo_ust10_mount prefix="${jackal_laser_mount}"
                           topic="${jackal_laser_topic}" />
-      <joint name="$(jackal_laser_mount)_laser_mount_joint" type="fixed">
-        <origin xyz="$(jackal_laser_offset)"
-                rpy="$(jackal_laser_rpy)" />
-        <parent link="$(jackal_laser_mount)_mount" />
-        <child link="$(jackal_laser_mount)_laser_mount" />
+      <joint name="${jackal_laser_mount}_laser_mount_joint" type="fixed">
+        <origin xyz="${jackal_laser_offset}"
+                rpy="${jackal_laser_rpy}" />
+        <parent link="${jackal_laser_mount}_mount" />
+        <child link="${jackal_laser_mount}_laser_mount" />
       </joint>
     </xacro:if>
-    <xacro:unless value="$(jackal_laser_hokuyo)">
+    <!--xacro:unless value="$(jackal_laser_hokuyo)">
       <xacro:include filename="$(find butler)/robots/jackal_description/urdf/accessories/sick_lms1xx_mount.urdf.xacro" />
       <sick_lms1xx_mount prefix="$(jackal_laser_mount)"
@@ -56,16 +40,16 @@
         <child link="$(jackal_laser_mount)_laser_mount" />
       </joint>
-    </xacro:unless>
+    </xacro:unless-->
   </xacro:if>
   <!-- If enabled, generate the upgraded Navsat payload (a Novatel Smart6). -->
-  <xacro:if value="$(jackal_navsat)">
+  <xacro:if value="${jackal_navsat}">
     <xacro:include filename="$(find butler)/robots/jackal_description/urdf/accessories/novatel_smart6.urdf.xacro" />
-    <bridge_plate mount="$(jackal_navsat_mount)"
-                  height="$(jackal_navsat_height)" />
-    <novatel_smart6 prefix="$(jackal_navsat_mount)"/>
-    <joint name="$(jackal_navsat_mount)_navsat_joint" type="fixed">
+    <bridge_plate mount="${jackal_navsat_mount}"
+                  height="${jackal_navsat_height}" />
+    <novatel_smart6 prefix="${jackal_navsat_mount}"/>
+    <joint name="${jackal_navsat_mount}_navsat_joint" type="fixed">
       <origin xyz="0 0 0" rpy="0 0 0" />
-      <parent link="$(jackal_navsat_mount)_bridge" />
-      <child link="$(jackal_navsat_mount)_navsat" />
+      <parent link="${jackal_navsat_mount}_bridge" />
+      <child link="${jackal_navsat_mount}_navsat" />
     </joint>
   </xacro:if>
@@ -141,16 +125,16 @@
     </joint>
   </xacro:if> -->
-  <xacro:if value="$(jackal_front_accessory_fender)">
+  <xacro:if value="${jackal_front_accessory_fender}">
     <xacro:include filename="$(find butler)/robots/jackal_description/urdf/accessories/hokuyo_ust10.urdf.xacro" />
-    <xacro:if value="$(jackal_front_fender_ust10)">
+    <xacro:if value="${jackal_front_fender_ust10}">
         <hokuyo_ust10 prefix="front_ust10" parent_link="front_fender_accessory_link"/>
     </xacro:if>
   </xacro:if>
-  <xacro:if value="$(jackal_rear_accessory_fender)">
-    <xacro:if value="$(jackal_rear_fender_ust10)">
+  <xacro:if value="${jackal_rear_accessory_fender}">
+    <xacro:if value="${jackal_rear_fender_ust10}">
         <hokuyo_ust10 prefix="rear_ust10" parent_link="rear_fender_accessory_link"/>
     </xacro:if>
   </xacro:if>
-  <xacro:if value="$(__JACKAL_ARK_ENCLOSURE)">
+  <xacro:if value="${__JACKAL_ARK_ENCLOSURE}">
     <link name="ark_enclosure_link">
       <visual>
@@ -171,3 +155,4 @@
     </gazebo>
   </xacro:if>
+  </xacro:macro>
 </robot>

File: robots/jackal_description/urdf/jackal.urdf.xacro (robot description, xacro)
@@ -228,5 +228,5 @@
   <xacro:arg name="jackal_laser_params" default=""/>
   <xacro:include filename="$(find butler)/robots/jackal_description/urdf/accessories.urdf.xacro" />
-  <xacro:read_model_data prefix="" config_jackal_file="${load_yaml('$(arg jackal_laser_params)')}"/>
+  <xacro:jackal prefix="" config_jackal_file="${load_yaml('$(arg jackal_laser_params)')}"/>
   <!-- Optional custom includes. -->
   <xacro:include filename="$(optenv JACKAL_URDF_EXTRAS empty.urdf)" />

Commit message: Added IMU and GPS plugins

File: robots/jackal_description/urdf/accessories.urdf.xacro (robot description, xacro)
@@ -54,4 +54,23 @@
     </joint>
   </xacro:if>
+<!--   Camera model integration -->
+<!--   <xacro:if value="$(optenv JACKAL_FLEA3 0)">
+  <camera_mount prefix="$(optenv JACKAL_FLEA3_MOUNT front)"
+                       tilt="$(optenv JACKAL_FLEA3_TILT 0.5236)"/>
+    <joint name="$(optenv JACKAL_FLEA3_MOUNT front)_camera_mount_joint" type="fixed">
+      <origin xyz="$(optenv JACKAL_FLEA3_OFFSET 0 0 0)"
+              rpy="$(optenv JACKAL_FLEA3_RPY 0 0 0)" />
+      <parent link="$(optenv JACKAL_FLEA3_MOUNT front)_mount" />
+      <child link="$(optenv JACKAL_FLEA3_MOUNT front)_camera_mount" />
+    </joint>
+    <pointgrey_flea3 frame="$(optenv JACKAL_FLEA3_MOUNT front)_camera" name="$(optenv JACKAL_FLEA3_NAME front)"
+      camera_x="0.0754" camera_y="0.029" camera_z="0.029"
+      camera_mass="0.085" hfov="1.0471975512" fps="60" width="640" height="512"/>
+    <joint name="$(optenv JACKAL_FLEA3_MOUNT front)_camera_bracket_joint" type="fixed">
+      <origin xyz="0.020 0 0.0245" rpy="0 0 0" />
+      <parent link="$(optenv JACKAL_FLEA3_MOUNT front)_camera_beam" />
+      <child link="$(optenv JACKAL_FLEA3_MOUNT front)_camera" />
+    </joint>
+  </xacro:if> -->
   <!-- Common camera mounts and accessory URDFs. -->
   <!-- <xacro:include filename="$(find butler)/robots/jackal_description/urdf/accessories/camera_mount.urdf.xacro" /> -->

Commit message: Added Laser Functionality

File: robots/jackal_description/urdf/accessories.urdf.xacro (robot description, xacro)
@@ -54,28 +54,9 @@
     </joint>
   </xacro:if>
-<!--   Camera model integration -->
+  <!-- Common camera mounts and accessory URDFs. -->
+ <!--  <xacro:include filename="$(find butler)/robots/jackal_description/urdf/accessories/camera_mount.urdf.xacro" />
+  <xacro:include filename="$(find pointgrey_camera_description)/urdf/pointgrey_flea3.urdf.xacro" /> -->
+  <!-- If enabled, generate the flea3 camera payload with a tilt of 30 degrees. -->
 <!--   <xacro:if value="$(optenv JACKAL_FLEA3 0)">
-  <camera_mount prefix="$(optenv JACKAL_FLEA3_MOUNT front)"
-                       tilt="$(optenv JACKAL_FLEA3_TILT 0.5236)"/>
-    <joint name="$(optenv JACKAL_FLEA3_MOUNT front)_camera_mount_joint" type="fixed">
-      <origin xyz="$(optenv JACKAL_FLEA3_OFFSET 0 0 0)"
-              rpy="$(optenv JACKAL_FLEA3_RPY 0 0 0)" />
-      <parent link="$(optenv JACKAL_FLEA3_MOUNT front)_mount" />
-      <child link="$(optenv JACKAL_FLEA3_MOUNT front)_camera_mount" />
-    </joint>
-    <pointgrey_flea3 frame="$(optenv JACKAL_FLEA3_MOUNT front)_camera" name="$(optenv JACKAL_FLEA3_NAME front)"
-      camera_x="0.0754" camera_y="0.029" camera_z="0.029"
-      camera_mass="0.085" hfov="1.0471975512" fps="60" width="640" height="512"/>
-    <joint name="$(optenv JACKAL_FLEA3_MOUNT front)_camera_bracket_joint" type="fixed">
-      <origin xyz="0.020 0 0.0245" rpy="0 0 0" />
-      <parent link="$(optenv JACKAL_FLEA3_MOUNT front)_camera_beam" />
-      <child link="$(optenv JACKAL_FLEA3_MOUNT front)_camera" />
-    </joint>
-  </xacro:if> -->
-  <!-- Common camera mounts and accessory URDFs. -->
-  <!-- <xacro:include filename="$(find butler)/robots/jackal_description/urdf/accessories/camera_mount.urdf.xacro" /> -->
-  <!-- <xacro:include filename="$(find pointgrey_camera_description)/urdf/pointgrey_flea3.urdf.xacro" /> -->
-  <!-- If enabled, generate the flea3 camera payload with a tilt of 30 degrees. -->
-  <!-- <xacro:if value="$(optenv JACKAL_FLEA3 0)">
     <camera_mount prefix="$(optenv JACKAL_FLEA3_MOUNT front)"
                        tilt="$(optenv JACKAL_FLEA3_TILT 0.5236)"/>
@@ -94,5 +75,6 @@
       <child link="$(optenv JACKAL_FLEA3_MOUNT front)_camera" />
     </joint>
-  </xacro:if> -->
+  </xacro:if>
+ -->
   <!-- <xacro:include filename="$(find butler)/robots/jackal_description/urdf/accessories/stereo_camera_mount.urdf.xacro" /> -->
   <!-- If enabled, generates a pair of flea3 cameras for stereo vision with a tilt of 30 degrees. -->

Commit message: Added Monocular Camera Configuration

File: robots/jackal_description/urdf/accessories.urdf.xacro (robot description, xacro)
@@ -55,26 +55,25 @@
   </xacro:if>
   <!-- Common camera mounts and accessory URDFs. -->
- <!--  <xacro:include filename="$(find butler)/robots/jackal_description/urdf/accessories/camera_mount.urdf.xacro" />
-  <xacro:include filename="$(find pointgrey_camera_description)/urdf/pointgrey_flea3.urdf.xacro" /> -->
+  <xacro:include filename="$(find butler)/robots/jackal_description/urdf/accessories/camera_mount.urdf.xacro" />
+  <xacro:include filename="$(find pointgrey_camera_description)/urdf/pointgrey_flea3.urdf.xacro" />
   <!-- If enabled, generate the flea3 camera payload with a tilt of 30 degrees. -->
-<!--   <xacro:if value="$(optenv JACKAL_FLEA3 0)">
-    <camera_mount prefix="$(optenv JACKAL_FLEA3_MOUNT front)"
-                       tilt="$(optenv JACKAL_FLEA3_TILT 0.5236)"/>
-    <joint name="$(optenv JACKAL_FLEA3_MOUNT front)_camera_mount_joint" type="fixed">
-      <origin xyz="$(optenv JACKAL_FLEA3_OFFSET 0 0 0)"
-              rpy="$(optenv JACKAL_FLEA3_RPY 0 0 0)" />
-      <parent link="$(optenv JACKAL_FLEA3_MOUNT front)_mount" />
-      <child link="$(optenv JACKAL_FLEA3_MOUNT front)_camera_mount" />
+  <xacro:if value="${jackal_flea3}">
+    <camera_mount prefix="${jackal_flea3_mount}"
+                       tilt="${jackal_flea3_tilt}"/>
+    <joint name="${jackal_flea3_mount}_camera_mount_joint" type="fixed">
+      <origin xyz="${jackal_flea3_offset}"
+              rpy="${jackal_flea3_rpy}" />
+      <parent link="${jackal_flea3_mount}_mount" />
+      <child link="${jackal_flea3_mount}_camera_mount" />
     </joint>
-    <pointgrey_flea3 frame="$(optenv JACKAL_FLEA3_MOUNT front)_camera" name="$(optenv JACKAL_FLEA3_NAME front)"
+    <pointgrey_flea3 frame="${jackal_flea3_mount}_camera" name="${jackal_flea3_name}"
       camera_x="0.0754" camera_y="0.029" camera_z="0.029"
       camera_mass="0.085" hfov="1.0471975512" fps="60" width="640" height="512"/>
-    <joint name="$(optenv JACKAL_FLEA3_MOUNT front)_camera_bracket_joint" type="fixed">
+    <joint name="${jackal_flea3_mount}_camera_bracket_joint" type="fixed">
       <origin xyz="0.020 0 0.0245" rpy="0 0 0" />
-      <parent link="$(optenv JACKAL_FLEA3_MOUNT front)_camera_beam" />
-      <child link="$(optenv JACKAL_FLEA3_MOUNT front)_camera" />
+      <parent link="${jackal_flea3_mount}_camera_beam" />
+      <child link="${jackal_flea3_mount}_camera" />
     </joint>
   </xacro:if>
- -->
   <!-- <xacro:include filename="$(find butler)/robots/jackal_description/urdf/accessories/stereo_camera_mount.urdf.xacro" /> -->
   <!-- If enabled, generates a pair of flea3 cameras for stereo vision with a tilt of 30 degrees. -->

File: robots/jackal_description/urdf/jackal.macro.xacro (robot description, xacro)
@@ -5,4 +5,5 @@
     <xacro:property name="__NAVSAT" value="${config_jackal_file['NAVSAT']}"/>
     <xacro:property name="__FENDER" value="${config_jackal_file['FENDER']}"/>
+    <xacro:property name="__FLEA3" value="${config_jackal_file['FLEA3']}"/>
     <xacro:property name="jackal_laser" value="${__LASER['JACKAL_LASER']}" scope="parent"/>
     <xacro:property name="jackal_laser_hokuyo" value="${__LASER['JACKAL_LASER_HOKUYO']}" scope="parent"/>
@@ -19,4 +20,10 @@
     <xacro:property name="jackal_rear_fender_ust10" value="${__FENDER['JACKAL_REAR_FENDER_UST10']}" scope="parent"/>
     <xacro:property name="__JACKAL_ARK_ENCLOSURE" value="${__FENDER['JACKAL_ARK_ENCLOSURE']}" scope="parent"/>
+    <xacro:property name="jackal_flea3" value="${__FLEA3['JACKAL_FLEA3']}" scope="parent"/>
+    <xacro:property name="jackal_flea3_mount" value="${__FLEA3['JACKAL_FLEA3_MOUNT']}" scope="parent"/>
+    <xacro:property name="jackal_flea3_tilt" value="${__FLEA3['JACKAL_FLEA3_TILT']}" scope="parent"/>
+    <xacro:property name="jackal_flea3_offset" value="${__FLEA3['JACKAL_FLEA3_OFFSET']}" scope="parent"/>
+    <xacro:property name="jackal_flea3_rpy" value="${__FLEA3['JACKAL_FLEA3_RPY']}" scope="parent"/>
+    <xacro:property name="jackal_flea3_name" value="${__FLEA3['JACKAL_FLEA3_NAME']}" scope="parent"/>
   </xacro:macro>
 </robot>
