Commit message: Added LiDAR configuration for Velodyne Puck

File: robots/jackal_description/urdf/accessories.urdf.xacro (robot description, xacro)
@@ -52,4 +52,27 @@
       <parent link="${jackal_navsat_mount}_bridge" />
       <child link="${jackal_navsat_mount}_navsat" />
+    </joint>
+  </xacro:if>
+  <!-- LiDAR integration parameters -->
+  <xacro:if value="${jackal_lidar == 1}">
+    <xacro:include filename="$(find butler)/robots/jackal_description/urdf/accessories/VLP-16.urdf.xacro"/>
+    <VLP-16 parent="front_mount" name="velodyne" topic="/velodyne_points">
+      <origin xyz="0 0 0.052" rpy="0 0 0" />
+    </VLP-16>
+    <link name="velodyne_mount">
+      <visual>
+        <origin xyz="0 0 0" rpy="0.0 0.0 0.0" />
+        <geometry>
+          <mesh filename="package://butler/robots/jackal_description/meshes/velodyne_mount.stl"/>
+        </geometry>
+        <material name="aluminum" >
+          <color rgba="0.45 0.45 0.45 1"/>
+        </material>
+      </visual>
+    </link>
+    <joint name="velodyne_mount_joint" type="fixed">
+      <parent link="velodyne_base_link" />
+      <child link="velodyne_mount" />
+      <origin xyz="0 0 0" />
     </joint>
   </xacro:if>

File: robots/jackal_description/urdf/jackal.macro.xacro (robot description, xacro)
@@ -6,4 +6,5 @@
     <xacro:property name="__FENDER" value="${config_jackal_file['FENDER']}"/>
     <xacro:property name="__FLEA3" value="${config_jackal_file['FLEA3']}"/>
+    <xacro:property name="__LIDAR" value="${config_jackal_file['LIDAR']}"/>
     <xacro:property name="jackal_laser" value="${__LASER['JACKAL_LASER']}" scope="parent"/>
     <xacro:property name="jackal_laser_hokuyo" value="${__LASER['JACKAL_LASER_HOKUYO']}" scope="parent"/>
@@ -26,4 +27,5 @@
     <xacro:property name="jackal_flea3_rpy" value="${__FLEA3['JACKAL_FLEA3_RPY']}" scope="parent"/>
     <xacro:property name="jackal_flea3_name" value="${__FLEA3['JACKAL_FLEA3_NAME']}" scope="parent"/>
+    <xacro:property name="jackal_lidar" value="${__LIDAR['JACKAL_LIDAR']}" scope="parent"/>
   </xacro:macro>
 </robot>
